File: kicad/esion-4aa.kicad_pcb (KiCad board)
At the start: 2 copper layers, 59.7 x 79 mm, 41 parts, among them Q1 BSS138, Q2 BSS192, SW4 POWER, U1 LM1117-3.3, U2 ESP32-WROOM, U3 ATtiny84-20SSU

Commit message: Добавлен сервер поискового индекса.
Parts:
- C2: value 100nF -> 0.1uF
- C3: value 0.1mF -> 0.1uF
- C4: value 100mF -> 10uF
- Q2: value BSS192 -> BSS192P
- R19: value R10K -> 10K
- moved C5 7.60 mm to (137.0, 78.9)
- moved R2 7.60 mm to (141.6, 78.9)
- moved Reset 7.60 mm to (150.2, 78.8)
- moved Configure 7.55 mm to (150.2, 71.2)
- moved R3 7.55 mm to (141.6, 71.2)
- renumbered Con.4 to Con.1, Con.3 to Con.2, Con.2 to Con.3, Con.1 to Con.4
Connections:
- BT1 pad 2: +3V3 -> Net-(BT1-Pad2)
- BT1 pad 4: +3V3 -> Net-(BT1-Pad2)
- BT2 pad 2: +3V3 -> Net-(BT1-Pad2)
- BT2 pad 4: +3V3 -> Net-(BT1-Pad2)
- C1 pad 1: Net-(C1-Pad1) -> M1
- D3 pad 1: Net-(C1-Pad1) -> M1
- Q2 pad 3: +6V -> M1
- Q2 pad 4: Net-(Q2-Pad2) -> (no net)
- R7 pad 1: +6V -> M1
- U1 pad 3: Net-(C1-Pad1) -> M1
Routing:
- net M1: track 0.00 -> 90.1 mm, vias 0 -> 2
- net +6V: track 115.2 -> 62.3 mm, vias 2 -> 1
- net +3V3: track 224.7 -> 177.0 mm
- net Net-(BT1-Pad2): track 15.2 -> 56.0 mm
- net Net-(C1-Pad1): track 16.4 -> 0.00 mm
- net Net-(J2-Pad5): track 106.2 -> 98.0 mm
- net GNDREF: track 271.8 -> 265.9 mm
- net Net-(R3-Pad2): track 37.1 -> 34.2 mm
Other:
- board text added: "+"
- board text added: "BT1"
- board text added: "BT2"
- board text added: "J2"
- board text added: "J5"
- board text added: "J6"
- board text added: "J7"
- board text added: "J8"
- board text added: "Q2"
- board text added: "SW1"
- board text added: "SW2"
- board text added: "U2"
- board text added: "_"
