File: kicad/esion-lo.kicad_pcb (KiCad board)
At the start: 2 copper layers, 89.1 x 33.1 mm, 41 parts, among them Q1 BSS138, Q2 BSS192, SW4 POWER, U1 AP2112K-3.3, U2 ESP32-WROOM, U3 ATtiny84-20SSU

Commit message: Добавлен сервер поискового индекса.
Parts:
- C2: value 100nF -> 0.1uF
- C3: value 0.1mF -> 0.1uF
- C4: value 10mF -> 10uF
- Conf.: value Configure -> SW2
- Q2: value BSS192 -> BSS192P
- R10: value 20k -> 20K
- R19: value R -> 10K
- Rst: value Reset -> SW1
Connections:
- C1 pad 1: Net-(C1-Pad1) -> M1
- D3 pad 1: Net-(C1-Pad1) -> M1
- Q2 pad 3: +3V8 -> M1
- Q2 pad 4: Net-(Q2-Pad2) -> (no net)
- R1 pad 1: Net-(C1-Pad1) -> M1
- R7 pad 1: +3V8 -> M1
- U1 pad 1: Net-(C1-Pad1) -> M1
Routing:
- net M1: track 0.00 -> 79.1 mm, vias 0 -> 3
- net +3V8: track 64.2 -> 20.9 mm, vias 3 -> 1
- net Net-(C1-Pad1): track 15.5 -> 0.00 mm
Other:
- board text added: "+"
- board text added: "J2"
- board text added: "J5"
- board text added: "J6"
- board text added: "J7"
- board text added: "J8"
- board text added: "Q2"
- board text added: "U2"
